Commit message: style(pre-commit): autofix

File: f1tenth/f1tenth_gym_ros/launch/ego_racecar.xacro (robot description, xacro)
@@ -2,14 +2,14 @@
 <!-- A simple model of the racecar for rviz -->
 <robot xmlns:xacro="http://www.ros.org/wiki/xacro" name="racecar">
-  <xacro:property name="wheelbase" value="0.3302" />
-  <xacro:property name="width" value="0.2032" />
-  <xacro:property name="height" value="0.1" />
-  <xacro:property name="ground_offset" value="0.04" />
-  <xacro:property name="wheel_radius" value="0.0508" />
-  <xacro:property name="wheel_length" value="0.0381" />
-  <xacro:property name="laser_distance_from_base_link" value="0.275" />
-  <xacro:property name="laser_height" value="0.05" />
-  <xacro:property name="laser_radius" value="0.026" />
-  <xacro:property name="car_name" value="ego_racecar" />
+  <xacro:property name="wheelbase" value="0.3302"/>
+  <xacro:property name="width" value="0.2032"/>
+  <xacro:property name="height" value="0.1"/>
+  <xacro:property name="ground_offset" value="0.04"/>
+  <xacro:property name="wheel_radius" value="0.0508"/>
+  <xacro:property name="wheel_length" value="0.0381"/>
+  <xacro:property name="laser_distance_from_base_link" value="0.275"/>
+  <xacro:property name="laser_height" value="0.05"/>
+  <xacro:property name="laser_radius" value="0.026"/>
+  <xacro:property name="car_name" value="ego_racecar"/>
   <material name="black">
     <color rgba="0.2 0.2 0.2 1."/>

File: f1tenth/f1tenth_gym_ros/launch/opp_racecar.xacro (robot description, xacro)
@@ -2,14 +2,14 @@
 <!-- A simple model of the racecar for rviz -->
 <robot xmlns:xacro="http://www.ros.org/wiki/xacro" name="racecar">
-  <xacro:property name="wheelbase" value="0.3302" />
-  <xacro:property name="width" value="0.2032" />
-  <xacro:property name="height" value="0.1" />
-  <xacro:property name="ground_offset" value="0.04" />
-  <xacro:property name="wheel_radius" value="0.0508" />
-  <xacro:property name="wheel_length" value="0.0381" />
-  <xacro:property name="laser_distance_from_base_link" value="0.275" />
-  <xacro:property name="laser_height" value="0.05" />
-  <xacro:property name="laser_radius" value="0.026" />
-  <xacro:property name="car_name" value="opp_racecar" />
+  <xacro:property name="wheelbase" value="0.3302"/>
+  <xacro:property name="width" value="0.2032"/>
+  <xacro:property name="height" value="0.1"/>
+  <xacro:property name="ground_offset" value="0.04"/>
+  <xacro:property name="wheel_radius" value="0.0508"/>
+  <xacro:property name="wheel_length" value="0.0381"/>
+  <xacro:property name="laser_distance_from_base_link" value="0.275"/>
+  <xacro:property name="laser_height" value="0.05"/>
+  <xacro:property name="laser_radius" value="0.026"/>
+  <xacro:property name="car_name" value="opp_racecar"/>
   <material name="black">
     <color rgba="0.2 0.2 0.2 1."/>
