Commit message: load sensors.xacro from individual_params
Signed-off-by: N-Eiki <eiki.nagata.2@tier4.jp>

File: launch/tier4_vehicle_launch/urdf/vehicle.xacro (robot description, xacro)
@@ -7,5 +7,4 @@
   <xacro:include filename="$(find ${vehicle_model_property}_description)/urdf/vehicle.xacro"/>
   <!-- sensors -->
-  <xacro:property name="sensor_model_property" value="$(arg sensor_model)"/>
-  <xacro:include filename="$(find ${sensor_model_property}_description)/urdf/sensors.xacro"/>
+  <xacro:include filename="$(find-pkg-share individual_params)/config/$(var vehicle_id)/urdf/sensors.xacro"/>
 </robot>
